File: hardware/main.kicad_sch (KiCad schematic)
At the start: 25 parts, among them J8101 KH-9752-6P6C, SW2 DM-04-V

Commit message: finish pcb
Parts:
- removed C52 (x2): 100n, Capacitor_SMD:C_0603_1608Metric, symbol Device:C_Small
- removed J?: MTB10-14S, Connector_IDC:IDC-Header_2x07_P2.54mm_Vertical, symbol Connector_Generic:Conn_02x07_Odd_Even
- removed SW2: DM-04-V, Button_Switch_SMD:SW_DIP_SPSTx04_Slide_6.7x11.72mm_W8.61mm_P2.54mm_LowProfile, symbol Switch:SW_DIP_x04
- added C? (x2): 100n, Capacitor_SMD:C_1206_3216Metric, symbol Device:C_Small
- added J15: DS1013-10S, Connector_IDC:IDC-Header_2x05_P2.54mm_Vertical, symbol Connector_Generic:Conn_02x05_Odd_Even
- added J8101: KH-9752-6P6C, MAS_Package_std:RJ12_Vertical, symbol Connector:RJ25
- J4: renamed from J?; footprint MAS_Package_nostd:AMASS_XT60-F_1x02_P7.20mm_Vertical -> MAS_Package_nostd:AMASS_XT60-M_1x02_P7.20mm_Vertical
- J8101: footprint MAS_Package_std:RJ12_Amphenol_54601 -> MAS_Package_std:RJ12_Vertical
- gave numbers to parts that had none: 3
Connections:
- net CANH: now also J8101.3, J15.7 (Pin_7), J8101.3
- net CANL: now also J8101.4, J15.8 (Pin_8), J8101.4
- net CANgnd: now also J8101.5, C?.2, J15.9 (Pin_9), J8101.5; no longer D5.1 (K)
- net CANvcc: now also J8101.2, C?.1, J15.10 (Pin_10), J8101.2; no longer R32.2
- net GND: now also D5.1 (K), J15.6 (Pin_6)
- net IO1: now also R32.2, J15.3 (Pin_3); no longer R32.2
- net IO2: now also R32.2, J15.4 (Pin_4); no longer R32.2
- net K1: now also SW2.1 (A), J15.1 (Pin_1)
- net K2: now also SW2.2 (B), J15.2 (Pin_2)
- net at J4.1: now also J3.1, J5.1, C?.1
- net at J4.2: now also J3.2, J5.2, C?.2
- new net IO3: J15.5 (Pin_5), R32.2
Other:
- moved on the sheet: J3, J4, J5, J8101, SW2

Commit message: Update main.kicad_sch
Other:
- company: (none) -> libreUPS
- title: (none) -> Communication panel board
Changed lines of the file:
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@@
   (paper "A5")
   (title_block
+    (title "Communication panel board")
     (date "2023-06-23")
     (rev "0.1")
+    (company "libreUPS")
+    (comment 2 "MuratovAS")
   )
   (junction (at 157.48 72.39) (diameter 0) (color 0 0 0 0)
